File: A2Pico.v2.6/A2Pico.v2.6.kicad_sch (KiCad schematic)
At the start: 27 parts, among them J1 Slide_Sw, J2 Conn_01x04, J3 Micro_SD_Card, J4 Apple2_slot, T1 2N7002, U1 RPI-Pico, U2 74LVC245, U3 74LVC245, U4 74LVC245, U5 74F11

Commit message: Add files via upload
Parts:
- removed T1: 2N7002, Package_TO_SOT_SMD:SOT-23, symbol Transistor_FET:2N7002
- added T1: 2N7000, Package_TO_SOT_THT:TO-92_Inline, symbol Transistor_FET:2N7000
Connections:
- net GND: now also T1.1 (S)
- net at J4.30 (~{IRQ}): now also T1.3 (D)
- net at R17.1, R17.2: now also T1.2 (G)
Changed lines of the file:
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@@
+	)
+	(symbol
+		(lib_id "Transistor_FET:2N7000")
+		(at 153.67 184.15 0)
+		(mirror y)
+		(unit 1)
+		(exclude_from_sim no)
+		(in_bom yes)
+		(on_board yes)
+		(dnp no)
+		(fields_autoplaced yes)
+		(property "Reference" "T1"
+			(at 147.32 182.8799 0)
+			(effects
+				(font
+					(size 1.27 1.27)
+				)
+				(justify left)
+			)
+		)
+		(property "Value" "2N7000"
+			(at 147.32 185.4199 0)
+			(effects
+				(font
+					(size 1.27 1.27)
+				)
+				(justify left)
+			)
+		)
+		(property "Footprint" "Package_TO_SOT_THT:TO-92_Inline"
+			(at 148.59 186.055 0)
+			(effects
+				(font
+					(size 1.27 1.27)
+					(italic yes)
+				)
+				(justify left)
+				(hide yes)
+			)
+		)
+		(property "Datasheet" "https://www.vishay.com/docs/70226/70226.pdf"
+			(at 148.59 187.96 0)
+			(effects
+				(font
+					(size 1.27 1.27)
+				)
+				(justify left)
+				(hide yes)
+			)
+		)
+		(property "Description" "0.2A Id, 200V Vds, N-Channel MOSFET, 2.6V Logic Level, TO-92"
+			(at 153.67 184.15 0)
+			(effects
+				(font
+					(size 1.27 1.27)
+				)
+				(hide yes)
+			)
+		)
+		(pin "2"
+		)
+		(pin "1"
+		)
+		(pin "3"
+		)
+		(instances
+			(project ""
+				(path "/eaef1172-3351-417c-bfc4-74a598f141cb"
+					(reference "T1")
+					(unit 1)
+				)
+			)
+		)
 	)
 	(symbol
@@
 					(unit 1)
 				)
-			)
-		)
-	)
-	(symbol
-		(lib_id "Transistor_FET:2N7002")
-		(at 153.67 184.15 0)
-		(mirror y)
-		(unit 1)
-		(exclude_from_sim no)
-		(in_bom yes)
-		(on_board yes)
-		(dnp no)
-		(fields_autoplaced yes)
-		(property "Reference" "T1"
-			(at 147.32 182.8799 0)
-			(effects
-				(font
-					(size 1.27 1.27)
-				)
-				(justify left)
-			)
-		)
-		(property "Value" "2N7002"
-			(at 147.32 185.4199 0)
-			(effects
-				(font
-					(size 1.27 1.27)
-				)
-				(justify left)
-			)
-		)
-		(property "Footprint" "Package_TO_SOT_SMD:SOT-23"
-			(at 148.59 186.055 0)
-			(effects
-				(font
-					(size 1.27 1.27)
-					(italic yes)
-				)
-				(justify left)
-				(hide yes)
-			)
-		)
-		(property "Datasheet" "https://www.onsemi.com/pub/Collateral/NDS7002A-D.PDF"
-			(at 148.59 187.96 0)
-			(effects
-				(font
-					(size 1.27 1.27)
-				)
-				(justify left)
-				(hide yes)
-			)
-		)
-		(property "Description" "0.115A Id, 60V Vds, N-Channel MOSFET, SOT-23"
-			(at 153.67 184.15 0)
-			(effects
-				(font
-					(size 1.27 1.27)
-				)
-				(hide yes)
-			)
-		)
-		(pin "1"
-		)
-		(pin "2"
-		)
-		(pin "3"
-		)
-		(instances
-			(project ""
-				(path "/eaef1172-3351-417c-bfc4-74a598f141cb"
-					(reference "T1")
-					(unit 1)
-				)

Commit message: Add files via upload
Other:
- note added: "1/8W"
Changed lines of the file:
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@@
+		)
+	)
+	(text "1/8W"
+		(exclude_from_sim no)
+		(at 175.26 48.514 0)
+		(effects
+			(font
+				(size 1.27 1.27)
+			)
+		)
+	)
+	(text "1/8W"
+		(exclude_from_sim no)
+		(at 159.766 51.054 0)
+		(effects
+			(font
+				(size 1.27 1.27)
+			)
+		)
+	)
+	(text "1/8W"
+		(exclude_from_sim no)
+		(at 165.354 189.992 0)
+		(effects
+			(font
+				(size 1.27 1.27)
+			)
+		)
+	)
+	(text "1/8W"
+		(exclude_from_sim no)
+		(at 166.37 186.69 0)
+		(effects
+			(font
+				(size 1.27 1.27)
+			)
+		)
+	)
+	(text "1/8W"
+		(exclude_from_sim no)
+		(at 102.616 17.78 0)
+		(effects
+			(font
+				(size 1.27 1.27)
+			)
 		)
 	)
@@
 		)
 		(property "Value" "+3V3"
-			(at 180.34 48.26 90)
+			(at 184.912 45.72 90)
 			(effects
 				(font
@@
 		(dnp no)
 		(property "Reference" "R17"
-			(at 102.87 17.78 90)
+			(at 102.87 13.208 90)
 			(effects
 				(font
@@
 		(dnp no)
 		(property "Reference" "R17"
-			(at 160.02 50.8 90)
+			(at 163.83 46.736 90)
 			(effects
 				(font
@@
 		)
 		(property "Value" "+3V3"
-			(at 165.1 50.8 90)
+			(at 166.116 50.038 90)
 			(effects
 				(font
@@
 		(dnp no)
 		(property "Reference" "R17"
-			(at 175.26 48.26 90)
-			(effects
-				(font
+			(at 175.26 43.434 90)
+			(effects
+				(font
